Commit message: gzaebo modified

File: alice_description/urdf/alice_robot.xacro (robot description, xacro)
@@ -15,5 +15,4 @@
   </joint>
 -->
-<!--
   <link name="base">
   </link>
@@ -23,5 +22,4 @@
     <child link="pelvis"/>
   </joint>
- -->
   <!-- pelvis -->
   <link name="pelvis">
@@ -62,5 +60,5 @@
     <child link="waist_pitch_link"/>
     <origin xyz="0 0 0.20" rpy="0 0 0"/>
-    <axis xyz="1 0 0"/>
+    <axis xyz="0 -1 0"/>
     <limit velocity="6.5" effort="1000" lower="${-pi/2}" upper="${pi}" />
     <dynamics damping = "0.7"/>
@@ -99,5 +97,5 @@
     <parent link="waist_pitch_link"/>
     <child link="waist_yaw_link"/>
-    <origin xyz="0 0 0.058" rpy="0 0 0"/>
+    <origin xyz="0 0 0.144" rpy="0 0 0"/>
     <axis xyz="0 0 -1"/>
     <limit velocity="6.5" effort="1000" lower="${-pi/2}" upper="${pi}" />
@@ -125,4 +123,109 @@
         <geometry>
           <mesh filename="package://alice_description/meshes/prt_robot_chest_3.stl" scale="0.001 0.001 0.001"/>
+        </geometry>
+        <material name="red"/>
+    </visual>
+    <inertial>
+      <origin xyz="0 0 0" rpy="0 0 0"/>
+      <mass value="1"/>
+      <inertia ixx="1.0" ixy="0.0" ixz="0.0" iyy="1.0" iyz="0.0" izz="1.0" />
+    </inertial>
+  </link>
+<!-- HEAD -->
+ <joint name="head_pitch" type="revolute">
+    <parent link="waist_yaw_link"/>
+    <child link="head_pitch_link"/>
+    <origin xyz="0 0 0.151" rpy="0 0 0"/>
+    <axis xyz="0 1 0"/>
+    <limit velocity="6.5" effort="1000" lower="${-pi/2}" upper="${pi}" />
+    <dynamics damping = "0.7"/>
+   </joint>
+  <transmission name="head_pitch_tran">
+     <type>transmission_interface/SimpleTransmission</type>
+     <joint name="head_pitch">
+       <hardwareInterface>EffortJointInterface</hardwareInterface>
+     </joint>
+     <actuator name="head_pitch_motor">
+       <hardwareInterface>EffortJointInterface</hardwareInterface>
+       <mechanicalReduction>1</mechanicalReduction>
+     </actuator>
+  </transmission>
+  <link name="head_pitch_link">
+    <collision>
+      <origin xyz="0 0 0" rpy="0 0 0"/>
+      <geometry>
+        <box size="0.01 0.01 0.01" />
+      </geometry>
+    </collision>
+    <visual>
+        <origin xyz="0 0 0" rpy="0 0 0"/>
+        <geometry>
+          <mesh filename="package://alice_description/meshes/prt_robot_head1.stl" scale="0.001 0.001 0.001"/>
+        </geometry>
+        <material name="red"/>
+    </visual>
+    <inertial>
+      <origin xyz="0 0 0" rpy="0 0 0"/>
+      <mass value="1"/>
+      <inertia ixx="1.0" ixy="0.0" ixz="0.0" iyy="1.0" iyz="0.0" izz="1.0" />
+    </inertial>
+  </link>
+ <joint name="head_yaw" type="revolute">
+    <parent link="head_pitch_link"/>
+    <child link="head_yaw_link"/>
+    <origin xyz="0 0 0.0875" rpy="0 0 0"/>
+    <axis xyz="0 0 1"/>
+    <limit velocity="6.5" effort="1000" lower="${-pi/2}" upper="${pi}" />
+    <dynamics damping = "0.7"/>
+   </joint>
+  <transmission name="head_yaw_tran">
+     <type>transmission_interface/SimpleTransmission</type>
+     <joint name="head_yaw">
+       <hardwareInterface>EffortJointInterface</hardwareInterface>
+     </joint>
+     <actuator name="head_yaw_motor">
+       <hardwareInterface>EffortJointInterface</hardwareInterface>
+       <mechanicalReduction>1</mechanicalReduction>
+     </actuator>
+  </transmission>
+  <link name="head_yaw_link">
+    <collision>
+      <origin xyz="0 0 0" rpy="0 0 0"/>
+      <geometry>
+        <box size="0.01 0.01 0.01" />
+      </geometry>
+    </collision>
+    <visual>
+        <origin xyz="0 0 0" rpy="0 0 0"/>
+        <geometry>
+          <mesh filename="package://alice_description/meshes/prt_robot_head2.stl" scale="0.001 0.001 0.001"/>
+        </geometry>
+        <material name="red"/>
+    </visual>
+    <inertial>
+      <origin xyz="0 0 0" rpy="0 0 0"/>
+      <mass value="1"/>
+      <inertia ixx="1.0" ixy="0.0" ixz="0.0" iyy="1.0" iyz="0.0" izz="1.0" />
+    </inertial>
+  </link>
+<joint name="camera_fixed" type="fixed">
+    <parent link="head_yaw_link"/>
+    <child link="camera_link"/>
+    <origin xyz="0.05 0 0.027" rpy="0 0 0"/>
+    <axis xyz="0 0 1"/>
+    <limit velocity="6.5" effort="1000" lower="${-pi/2}" upper="${pi}" />
+    <dynamics damping = "0.7"/>
+ </joint>
+  <link name="camera_link">
+    <collision>
+      <origin xyz="0 0 0" rpy="0 0 0"/>
+      <geometry>
+        <box size="0.01 0.01 0.01" />
+      </geometry>
+    </collision>
+    <visual>
+        <origin xyz="0 0 0" rpy="0 0 0"/>
+        <geometry>
+          <mesh filename="package://alice_description/meshes/prt_zed_camera_simul.stl" scale="0.001 0.001 0.001"/>
         </geometry>
         <material name="red"/>
@@ -561,5 +664,5 @@
     <child link="l_hip_yaw_link"/>
     <origin xyz="0 0 -0.136" rpy="0 0 0"/>
-    <axis xyz="0 0 -1"/>
+    <axis xyz="0 0 1"/>
     <limit velocity="6.5" effort="1000" lower="${-pi/2}" upper="${pi/2}" />
     <dynamics damping = "0.7"/>
@@ -771,5 +874,5 @@
     <child link="r_hip_roll_link"/>
     <origin xyz="0 -0.056 0" rpy="0 0 0"/>
-    <axis xyz="-1 0 0"/>
+    <axis xyz="1 0 0"/>
     <limit velocity="6.5" effort="1000" lower="${-pi}" upper="${pi/2}" />
     <dynamics damping = "0.7"/>
@@ -810,5 +913,5 @@
     <child link="r_hip_yaw_link"/>
     <origin xyz="0 0 -0.136" rpy="0 0 0"/>
-    <axis xyz="0 0 -1"/>
+    <axis xyz="0 0 1"/>
     <limit velocity="6.5" effort="1000" lower="${-pi/2}" upper="${pi/2}" />
     <dynamics damping = "0.7"/>

Commit message: gazebo urdf modified

File: alice_description/urdf/alice_robot.xacro (robot description, xacro)
@@ -60,5 +60,5 @@
     <child link="waist_pitch_link"/>
     <origin xyz="0 0 0.20" rpy="0 0 0"/>
-    <axis xyz="0 -1 0"/>
+    <axis xyz="0 1 0"/>
     <limit velocity="6.5" effort="1000" lower="${-pi/2}" upper="${pi}" />
     <dynamics damping = "0.7"/>
@@ -98,5 +98,5 @@
     <child link="waist_yaw_link"/>
     <origin xyz="0 0 0.144" rpy="0 0 0"/>
-    <axis xyz="0 0 -1"/>
+    <axis xyz="0 0 1"/>
     <limit velocity="6.5" effort="1000" lower="${-pi/2}" upper="${pi}" />
     <dynamics damping = "0.7"/>
@@ -237,350 +237,4 @@
     </inertial>
   </link>
-  <!-- head
-  <joint name="head_yaw" type="revolute">
-    <parent link="waist_yaw_link"/>
-    <child link="head_yaw_link"/>
-    <origin xyz="0 0 0.1935" rpy="0 0 0"/>
-    <axis xyz="0 0 -1"/>
-    <limit velocity="6.5" effort="1000" lower="${-pi/2}" upper="${pi/2}" />
-    <dynamics damping = "0.7"/>
-  </joint>
-  <transmission name="head_yaw_tran">
-     <type>transmission_interface/SimpleTransmission</type>
-     <joint name="head_yaw">
-       <hardwareInterface>EffortJointInterface</hardwareInterface>
-     </joint>
-     <actuator name="head_yaw_motor">
-       <hardwareInterface>EffortJointInterface</hardwareInterface>
-       <mechanicalReduction>1</mechanicalReduction>
-     </actuator>
-  </transmission>
-  <link name="head_yaw_link">
-    <collision>
-      <origin xyz="0 0 0" rpy="0 0 0"/>
-      <geometry>
-        <box size="0.01 0.01 0.01" />
-      </geometry>
-    </collision>
-    <visual>
-        <origin xyz="0 0 0" rpy="0 0 0"/>
-        <geometry>
-          <mesh filename="package://diana_description/meshes/stl_robot_head1.stl" scale="0.001 0.001 0.001"/>
-        </geometry>
-        <material name="red"/>
-    </visual>
-    <inertial>
-      <origin xyz="0 0 0" rpy="0 0 0"/>
-      <mass value="1"/>
-      <inertia ixx="1.0" ixy="0.0" ixz="0.0" iyy="1.0" iyz="0.0" izz="1.0" />
-    </inertial>
-  </link>
-  <joint name="head_pitch" type="revolute">
-    <parent link="head_yaw_link"/>
-    <child link="head_pitch_link"/>
-    <origin xyz="0 0 0.095" rpy="0 0 0"/>
-    <axis xyz="0 -1 0"/>
-    <limit velocity="6.5" effort="1000" lower="${-pi/2}" upper="${pi/2}" />
-    <dynamics damping = "0.7"/>
-  </joint>
-  <transmission name="head_pitch_tran">
-     <type>transmission_interface/SimpleTransmission</type>
-     <joint name="head_pitch">
-       <hardwareInterface>EffortJointInterface</hardwareInterface>
-     </joint>
-     <actuator name="head_pitch_motor">
-       <hardwareInterface>EffortJointInterface</hardwareInterface>
-       <mechanicalReduction>1</mechanicalReduction>
-     </actuator>
-   </transmission>
-  <link name="head_pitch_link">
-    <collision>
-      <origin xyz="0 0 0" rpy="0 0 0"/>
-      <geometry>
-        <box size="0.01 0.01 0.01" />
-      </geometry>
-    </collision>
-    <visual>
-        <origin xyz="0 0 0" rpy="0 0 0"/>
-        <geometry>
-          <mesh filename="package://diana_description/meshes/stl_robot_head2.stl" scale="0.001 0.001 0.001"/>
-        </geometry>
-        <material name="red"/>
-    </visual>
-    <inertial>
-      <origin xyz="0 0 0" rpy="0 0 0"/>
-      <mass value="1"/>
-      <inertia ixx="1.0" ixy="0.0" ixz="0.0" iyy="1.0" iyz="0.0" izz="1.0" />
-    </inertial>
-  </link>
-  <joint name="head_roll" type="revolute">
-    <parent link="head_pitch_link"/>
-    <child link="head_roll_link"/>
-    <origin xyz="0 0 0" rpy="0 0 0"/>
-    <axis xyz="-1 0 0"/>
-    <limit velocity="6.5" effort="1000" lower="${-pi/2}" upper="${pi/2}" />
-    <dynamics damping = "0.7"/>
-  </joint>
-  <transmission name="head_roll_tran">
-     <type>transmission_interface/SimpleTransmission</type>
-     <joint name="head_roll">
-       <hardwareInterface>EffortJointInterface</hardwareInterface>
-     </joint>
-     <actuator name="head_roll_motor">
-       <hardwareInterface>EffortJointInterface</hardwareInterface>
-       <mechanicalReduction>1</mechanicalReduction>
-     </actuator>
-  </transmission>
-  <link name="head_roll_link">
-    <collision>
-      <origin xyz="0 0 0" rpy="0 0 0"/>
-      <geometry>
-        <box size="0.01 0.01 0.01" />
-      </geometry>
-    </collision>
-    <visual>
-        <origin xyz="0 0 0" rpy="0 0 0"/>
-        <geometry>
-          <mesh filename="package://diana_description/meshes/stl_robot_head3.stl" scale="0.001 0.001 0.001"/>
-        </geometry>
-        <material name="red"/>
-    </visual>
-    <inertial>
-      <origin xyz="0 0 0" rpy="0 0 0"/>
-      <mass value="1"/>
-      <inertia ixx="1.0" ixy="0.0" ixz="0.0" iyy="1.0" iyz="0.0" izz="1.0" />
-    </inertial>
-  </link>
-   left Arm
-  <joint name="l_shoulder_pitch" type="revolute">
-    <parent link="waist_yaw_link"/>
-    <child link="l_shoulder_pitch_link"/>
-    <origin xyz="0 0.1535 0.147" rpy="0 0 0"/>
-    <axis xyz="0 -1 0"/>
-    <limit velocity="6.5" effort="1000" lower="${-pi/2}" upper="${pi}" />
-    <dynamics damping = "0.7"/>
-  </joint>
-  <transmission name="l_shoulder_pitch_tran">
-     <type>transmission_interface/SimpleTransmission</type>
-     <joint name="l_shoulder_pitch">
-       <hardwareInterface>EffortJointInterface</hardwareInterface>
-     </joint>
-     <actuator name="l_shoulder_pitch_motor">
-       <hardwareInterface>EffortJointInterface</hardwareInterface>
-       <mechanicalReduction>1</mechanicalReduction>
-     </actuator>
-  </transmission>
-  <link name="l_shoulder_pitch_link">
-    <collision>
-      <origin xyz="0 0 0" rpy="0 0 0"/>
-      <geometry>
-        <box size="0.01 0.01 0.01" />
-      </geometry>
-    </collision>
-    <visual>
-        <origin xyz="0 0 0" rpy="0 0 0"/>
-        <geometry>
-          <mesh filename="package://diana_description/meshes/stl_robot_arm_left1.stl" scale="0.001 0.001 0.001"/>
-        </geometry>
-        <material name="red"/>
-    </visual>
-    <inertial>
-      <origin xyz="0 0 0" rpy="0 0 0"/>
-      <mass value="1"/>
-      <inertia ixx="1.0" ixy="0.0" ixz="0.0" iyy="1.0" iyz="0.0" izz="1.0" />
-    </inertial>
-  </link>
-  <joint name="l_shoulder_roll" type="revolute">
-    <parent link="l_shoulder_pitch_link"/>
-    <child link="l_shoulder_roll_link"/>
-    <origin xyz="0 0.0515 0" rpy="-1.570796327 0 0"/>
-    <axis xyz="-1 0 0"/>
-    <limit velocity="6.5" effort="1000" lower="${-pi/2}" upper="${pi}" />
-    <dynamics damping = "0.7"/>
-  </joint>
-  <transmission name="l_shoulder_roll_tran">
-     <type>transmission_interface/SimpleTransmission</type>
-     <joint name="l_shoulder_roll">
-       <hardwareInterface>EffortJointInterface</hardwareInterface>
-     </joint>
-     <actuator name="l_shoulder_roll_motor">
-       <hardwareInterface>EffortJointInterface</hardwareInterface>
-       <mechanicalReduction>1</mechanicalReduction>
-     </actuator>
-  </transmission>
-  <link name="l_shoulder_roll_link">
-    <collision>
-      <origin xyz="0 0 0" rpy="0 0 0"/>
-      <geometry>
-        <box size="0.01 0.01 0.01" />
-      </geometry>
-    </collision>
-    <visual>
-        <origin xyz="0 0 0" rpy="0 0 0"/>
-        <geometry>
-          <mesh filename="package://diana_description/meshes/stl_robot_arm_left2.stl" scale="0.001 0.001 0.001"/>
-        </geometry>
-        <material name="red"/>
-    </visual>
-    <inertial>
-      <origin xyz="0 0 0" rpy="0 0 0"/>
-      <mass value="1"/>
-      <inertia ixx="1.0" ixy="0.0" ixz="0.0" iyy="1.0" iyz="0.0" izz="1.0" />
-    </inertial>
-  </link>
-  <joint name="l_elbow_pitch" type="revolute">
-    <parent link="l_shoulder_roll_link"/>
-    <child link="l_elbow_pitch_link"/>
-    <origin xyz="0 0.2 0" rpy="0 0 0"/>
-    <axis xyz="0 0 1"/>
-    <limit velocity="6.5" effort="1000" lower="${-pi/2}" upper="${pi/2}" />
-    <dynamics damping = "0.7"/>
-  </joint>
-  <transmission name="l_elbow_pitch_tran">
-     <type>transmission_interface/SimpleTransmission</type>
-     <joint name="l_elbow_pitch">
-       <hardwareInterface>EffortJointInterface</hardwareInterface>
-     </joint>
-     <actuator name="l_elbow_pitch_motor">
-       <hardwareInterface>EffortJointInterface</hardwareInterface>
-       <mechanicalReduction>1</mechanicalReduction>
-     </actuator>
-  </transmission>
-  <link name="l_elbow_pitch_link">
-    <collision>
-      <origin xyz="0 0 0" rpy="0 0 0"/>
-      <geometry>
-        <box size="0.01 0.01 0.01" />
-      </geometry>
-    </collision>
-    <visual>
-        <origin xyz="0 0 0" rpy="0 0 0"/>
-        <geometry>
-          <mesh filename="package://diana_description/meshes/stl_robot_arm_left3.stl" scale="0.001 0.001 0.001"/>
-        </geometry>
-        <material name="red"/>
-    </visual>
-    <inertial>
-      <origin xyz="0 0 0" rpy="0 0 0"/>
-      <mass value="1"/>
-      <inertia ixx="1.0" ixy="0.0" ixz="0.0" iyy="1.0" iyz="0.0" izz="1.0" />
-    </inertial>
-  </link>
-   right Arm
-  <joint name="r_shoulder_pitch" type="revolute">
-    <parent link="waist_yaw_link"/>
-    <child link="r_shoulder_pitch_link"/>
-    <origin xyz="0 -0.1535 0.147" rpy="0 0 0"/>
-    <axis xyz="0 1 0"/>
-    <limit velocity="6.5" effort="1000" lower="${-pi/2}" upper="${pi}" />
-    <dynamics damping = "0.7"/>
-  </joint>
-  <transmission name="r_shoulder_pitch_tran">
-     <type>transmission_interface/SimpleTransmission</type>
-     <joint name="r_shoulder_pitch">
-       <hardwareInterface>EffortJointInterface</hardwareInterface>
-     </joint>
-     <actuator name="r_shoulder_pitch_motor">
-       <hardwareInterface>EffortJointInterface</hardwareInterface>
-       <mechanicalReduction>1</mechanicalReduction>
-     </actuator>
-  </transmission>
-  <link name="r_shoulder_pitch_link">
-    <collision>
-      <origin xyz="0 0 0" rpy="0 0 0"/>
-      <geometry>
-        <box size="0.01 0.01 0.01" />
-      </geometry>
-    </collision>
-    <visual>
-        <origin xyz="0 0 0" rpy="0 0 0"/>
-        <geometry>
-          <mesh filename="package://diana_description/meshes/stl_robot_arm_right1.stl" scale="0.001 0.001 0.001"/>
-        </geometry>
-        <material name="red"/>
-    </visual>
-    <inertial>
-      <origin xyz="0 0 0" rpy="0 0 0"/>
-      <mass value="1"/>
-      <inertia ixx="1.0" ixy="0.0" ixz="0.0" iyy="1.0" iyz="0.0" izz="1.0" />
-    </inertial>
-  </link>
-  <joint name="r_shoulder_roll" type="revolute">
-    <parent link="r_shoulder_pitch_link"/>
-    <child link="r_shoulder_roll_link"/>
-    <origin xyz="0 -0.0515 0" rpy="1.570796327 0 0"/>
-    <axis xyz="-1 0 0"/>
-    <limit velocity="6.5" effort="1000" lower="${-pi/2}" upper="${pi}" />
-    <dynamics damping = "0.7"/>
-  </joint>
-  <transmission name="r_shoulder_roll_tran">
-     <type>transmission_interface/SimpleTransmission</type>
-     <joint name="r_shoulder_roll">
-       <hardwareInterface>EffortJointInterface</hardwareInterface>
-     </joint>
-     <actuator name="r_shoulder_roll_motor">
-       <hardwareInterface>EffortJointInterface</hardwareInterface>
-       <mechanicalReduction>1</mechanicalReduction>
-     </actuator>
-  </transmission>
-  <link name="r_shoulder_roll_link">
-    <collision>
-      <origin xyz="0 0 0" rpy="0 0 0"/>
-      <geometry>
-        <box size="0.01 0.01 0.01" />
-      </geometry>
-    </collision>
-    <visual>
-        <origin xyz="0 0 0" rpy="0 0 0"/>
-        <geometry>
-          <mesh filename="package://diana_description/meshes/stl_robot_arm_right2.stl" scale="0.001 0.001 0.001"/>
-        </geometry>
-        <material name="red"/>
-    </visual>
-    <inertial>
-      <origin xyz="0 0 0" rpy="0 0 0"/>
-      <mass value="1"/>
-      <inertia ixx="1.0" ixy="0.0" ixz="0.0" iyy="1.0" iyz="0.0" izz="1.0" />
-    </inertial>
-  </link>
-  <joint name="r_elbow_pitch" type="revolute">
-    <parent link="r_shoulder_roll_link"/>
-    <child link="r_elbow_pitch_link"/>
-    <origin xyz="0 -0.2 0" rpy="0 0 0"/>
-    <axis xyz="0 0 1"/>
-    <limit velocity="6.5" effort="1000" lower="${-pi/2}" upper="${pi/2}" />
-    <dynamics damping = "0.7"/>
-  </joint>
-  <transmission name="r_elbow_pitch_tran">
-     <type>transmission_interface/SimpleTransmission</type>
-     <joint name="r_elbow_pitch">
-       <hardwareInterface>EffortJointInterface</hardwareInterface>
-     </joint>
-     <actuator name="r_elbow_pitch_motor">
-       <hardwareInterface>EffortJointInterface</hardwareInterface>
-       <mechanicalReduction>1</mechanicalReduction>
-     </actuator>
-  </transmission>
-  <link name="r_elbow_pitch_link">
-    <collision>
-      <origin xyz="0 0 0" rpy="0 0 0"/>
-      <geometry>
-        <box size="0.01 0.01 0.01" />
-      </geometry>
-    </collision>
-    <visual>
-        <origin xyz="0 0 0" rpy="0 0 0"/>
-        <geometry>
-          <mesh filename="package://diana_description/meshes/stl_robot_arm_right3.stl" scale="0.001 0.001 0.001"/>
-        </geometry>
-        <material name="red"/>
-    </visual>
-    <inertial>
-      <origin xyz="0 0 0" rpy="0 0 0"/>
-      <mass value="1"/>
-      <inertia ixx="1.0" ixy="0.0" ixz="0.0" iyy="1.0" iyz="0.0" izz="1.0" />
-    </inertial>
-  </link>
--->
   <!-- left leg -->
   <joint name="l_hip_pitch" type="revolute">
@@ -588,5 +242,5 @@
     <child link="l_hip_pitch_link"/>
     <origin xyz="0 0.034 0" rpy="0 0 0"/>
-    <axis xyz="0 -1 0"/>
+    <axis xyz="0 1 0"/>
     <limit velocity="6.5" effort="1000" lower="${-pi/2}" upper="${pi/2}" />
     <dynamics damping = "0.7"/>
@@ -626,5 +280,5 @@
     <child link="l_hip_roll_link"/>
     <origin xyz="0 0.056 0" rpy="0 0 0"/>
-    <axis xyz="-1 0 0"/>
+    <axis xyz="1 0 0"/>
     <limit velocity="6.5" effort="1000" lower="${-pi/2}" upper="${pi}" />
     <dynamics damping = "0.7"/>
@@ -702,5 +356,5 @@
     <child link="l_knee_pitch_link"/>
     <origin xyz="0 0 -0.104" rpy="0 0 0"/>
-    <axis xyz="0 -1 0"/>
+    <axis xyz="0 1 0"/>
     <limit velocity="6.5" effort="1000" lower="${-pi}" upper="${pi/2}" />
     <dynamics damping = "0.7"/>
@@ -991,5 +645,5 @@
     <child link="r_ankle_pitch_link"/>
     <origin xyz="0 0 -0.240" rpy="0 0 0"/>
-    <axis xyz="0 -1 0"/>
+    <axis xyz="0 1 0"/>
     <limit velocity="6.5" effort="1000" lower="${-pi/2}" upper="${pi/2}" />
     <dynamics damping = "0.7"/>

Commit message: urdf modified

File: alice_description/urdf/alice_robot.xacro (robot description, xacro)
@@ -18,5 +18,5 @@
   </link>
   <joint name="base_fixed" type="fixed">
-    <origin xyz="0 0 0.7" rpy="0 0 0"/>
+    <origin xyz="0 0 0.57" rpy="0 0 0"/>
     <parent link="base"/>
     <child link="pelvis"/>
@@ -60,5 +60,5 @@
     <child link="waist_pitch_link"/>
     <origin xyz="0 0 0.20" rpy="0 0 0"/>
-    <axis xyz="0 1 0"/>
+    <axis xyz="0 -1 0"/>
     <limit velocity="6.5" effort="1000" lower="${-pi/2}" upper="${pi}" />
     <dynamics damping = "0.7"/>
@@ -98,5 +98,5 @@
     <child link="waist_yaw_link"/>
     <origin xyz="0 0 0.144" rpy="0 0 0"/>
-    <axis xyz="0 0 1"/>
+    <axis xyz="0 0 -1"/>
     <limit velocity="6.5" effort="1000" lower="${-pi/2}" upper="${pi}" />
     <dynamics damping = "0.7"/>
@@ -242,5 +242,5 @@
     <child link="l_hip_pitch_link"/>
     <origin xyz="0 0.034 0" rpy="0 0 0"/>
-    <axis xyz="0 1 0"/>
+    <axis xyz="0 -1 0"/>
     <limit velocity="6.5" effort="1000" lower="${-pi/2}" upper="${pi/2}" />
     <dynamics damping = "0.7"/>
@@ -280,5 +280,5 @@
     <child link="l_hip_roll_link"/>
     <origin xyz="0 0.056 0" rpy="0 0 0"/>
-    <axis xyz="1 0 0"/>
+    <axis xyz="-1 0 0"/>
     <limit velocity="6.5" effort="1000" lower="${-pi/2}" upper="${pi}" />
     <dynamics damping = "0.7"/>
@@ -356,5 +356,5 @@
     <child link="l_knee_pitch_link"/>
     <origin xyz="0 0 -0.104" rpy="0 0 0"/>
-    <axis xyz="0 1 0"/>
+    <axis xyz="0 -1 0"/>
     <limit velocity="6.5" effort="1000" lower="${-pi}" upper="${pi/2}" />
     <dynamics damping = "0.7"/>
@@ -528,5 +528,5 @@
     <child link="r_hip_roll_link"/>
     <origin xyz="0 -0.056 0" rpy="0 0 0"/>
-    <axis xyz="1 0 0"/>
+    <axis xyz="-1 0 0"/>
     <limit velocity="6.5" effort="1000" lower="${-pi}" upper="${pi/2}" />
     <dynamics damping = "0.7"/>
@@ -645,5 +645,5 @@
     <child link="r_ankle_pitch_link"/>
     <origin xyz="0 0 -0.240" rpy="0 0 0"/>
-    <axis xyz="0 1 0"/>
+    <axis xyz="0 -1 0"/>
     <limit velocity="6.5" effort="1000" lower="${-pi/2}" upper="${pi/2}" />
     <dynamics damping = "0.7"/>
