Commit message: model modified

File: alice_1_description/urdf/alice_1_robot.xacro (robot description, xacro)
@@ -194,7 +194,7 @@
 <!-- l_shoulder_pitch -->
   <joint name="l_shoulder_pitch" type="revolute">
-    <parent link="head_pitch_link"/>
+    <parent link="pelvis_waist"/>
     <child link="l_shoulder_pitch_link"/>
-    <origin xyz="0 0.17 -0.0565" rpy="0 0 0"/>
+    <origin xyz="0 0.17 0.4100" rpy="0 0 0"/>
     <axis xyz="0 1 0"/>
     <limit velocity="6.5" effort="1000" lower="${-pi/2}" upper="${pi}" />
@@ -233,7 +233,7 @@
 <!-- r_shoulder_pitch -->
  <joint name="r_shoulder_pitch" type="revolute">
-    <parent link="head_pitch_link"/>
+    <parent link="pelvis_waist"/>
     <child link="r_shoulder_pitch_link"/>
-    <origin xyz="0 -0.17 -0.0565" rpy="0 0 0"/>
+    <origin xyz="0 -0.17 0.4100" rpy="0 0 0"/>
     <axis xyz="0 1 0"/>
     <limit velocity="6.5" effort="1000" lower="${-pi/2}" upper="${pi}" />
@@ -746,13 +746,31 @@
   <joint name="imu_fixed" type="fixed">
     <parent link="pelvis_waist"/>
-    <child link="imu_link"/>
-    <origin xyz="0.0 0.0 0" rpy="0 0 0"/>
-  </joint>
-  <link name="imu_link">
-    <inertial>
-      <origin xyz="0 0 0" rpy="0 0 0"/>
-      <mass value="0"/>
-      <inertia ixx="1.0" ixy="0.0" ixz="0.0" iyy="1.0" iyz="0.0" izz="1.0" />
-    </inertial>
-  </link>
+    <child link="imu_link_1"/>
+    <origin xyz="0 0 0" rpy="0 0 -1.57079632679"/>
+  </joint>
+  <link name="imu_link_1">
+    <collision>
+      <origin xyz="0 0 0" rpy="0 0 0"/>
+      <geometry>
+        <box size="0.01 0.01 0.01" />
+      </geometry>
+    </collision>
+    <inertial>
+      <origin xyz="0 0 0" rpy="0 0 0"/>
+      <mass value="0.1"/>
+      <inertia ixx="1.0" ixy="0.0" ixz="0.0" iyy="1.0" iyz="0.0" izz="1.0" />
+    </inertial>
+  </link>
+  <joint name="imu_fixed_1" type="fixed">
+    <parent link="imu_link_1"/>
+    <child link="imu_link_2"/>
+    <origin xyz="0 0 0" rpy="0 3.1415926535 0"/>
+  </joint>
+   <link name="imu_link_2">
+    <inertial>
+      <origin xyz="0 0 0" rpy="0 0 0"/>
+      <mass value="0.1"/>
+      <inertia ixx="1.0" ixy="0.0" ixz="0.0" iyy="1.0" iyz="0.0" izz="1.0" />
+    </inertial>
+   </link>
 </robot>

File: alice_2_description/urdf/alice_2_robot.xacro (robot description, xacro)
@@ -101,4 +101,16 @@
     </inertial>
   </link>
+<joint name="camera_zed" type="fixed">
+    <parent link="head_fixed"/>
+    <child link="camera_zed_link"/>
+    <origin xyz="0.1 0.0 0" rpy="0 0 0"/>
+  </joint>
+  <link name="camera_zed_link">
+    <inertial>
+      <origin xyz="0 0 0" rpy="0 0 0"/>
+      <mass value="0"/>
+      <inertia ixx="1.0" ixy="0.0" ixz="0.0" iyy="1.0" iyz="0.0" izz="1.0" />
+    </inertial>
+  </link>
 <!-- left_leg -->
   <joint name="pelvis_pitch_l" type="revolute">

Commit message: model_modified

File: alice_1_description/urdf/alice_1_robot.xacro (robot description, xacro)
@@ -271,7 +271,7 @@
   </link>
 <!-- left_leg -->
-  <joint name="pelvis_pitch_l" type="revolute">
+  <joint name="l_hip_pitch" type="revolute">
     <parent link="pelvis_waist"/>
-    <child link="pelvis_l1"/>
+    <child link="l_hip_pitch_link"/>
     <origin xyz="0 0.021 0" rpy="0 0 0"/>
     <axis xyz="0 -1 0"/>
@@ -279,15 +279,15 @@
     <dynamics damping = "0.7"/>
   </joint>
-  <transmission name="pelvis_pitch_l_tran">
-     <type>transmission_interface/SimpleTransmission</type>
-     <joint name="pelvis_pitch_l">
-       <hardwareInterface>EffortJointInterface</hardwareInterface>
-     </joint>
-     <actuator name="pelvis_pitch_l_motor">
-       <hardwareInterface>EffortJointInterface</hardwareInterface>
-       <mechanicalReduction>1</mechanicalReduction>
-     </actuator>
-  </transmission>
-  <link name="pelvis_l1">
+  <transmission name="l_hip_pitch_tran">
+     <type>transmission_interface/SimpleTransmission</type>
+     <joint name="l_hip_pitch">
+       <hardwareInterface>EffortJointInterface</hardwareInterface>
+     </joint>
+     <actuator name="l_hip_pitch_motor">
+       <hardwareInterface>EffortJointInterface</hardwareInterface>
+       <mechanicalReduction>1</mechanicalReduction>
+     </actuator>
+  </transmission>
+  <link name="l_hip_pitch_link">
     <collision>
       <origin xyz="0 0 0" rpy="0 0 0"/>
@@ -309,7 +309,7 @@
     </inertial>
   </link>
-  <joint name="pelvis_roll_l" type="revolute">
-    <parent link="pelvis_l1"/>
-    <child link="pelvis_l2"/>
+  <joint name="l_hip_roll" type="revolute">
+    <parent link="l_hip_pitch_link"/>
+    <child link="l_hip_roll_link"/>
     <origin xyz="0 0.059 0" rpy="0 0 0"/>
     <axis xyz="-1 0 0"/>
@@ -317,15 +317,15 @@
     <dynamics damping = "0.7"/>
   </joint>
-  <transmission name="pelvis_roll_l_tran">
-     <type>transmission_interface/SimpleTransmission</type>
-     <joint name="pelvis_roll_l">
-       <hardwareInterface>EffortJointInterface</hardwareInterface>
-     </joint>
-     <actuator name="pelvis_roll_l_motor">
-       <hardwareInterface>EffortJointInterface</hardwareInterface>
-       <mechanicalReduction>1</mechanicalReduction>
-     </actuator>
-  </transmission>
-   <link name="pelvis_l2">
+  <transmission name="l_hip_roll_tran">
+     <type>transmission_interface/SimpleTransmission</type>
+     <joint name="l_hip_roll">
+       <hardwareInterface>EffortJointInterface</hardwareInterface>
+     </joint>
+     <actuator name="l_hip_roll_motor">
+       <hardwareInterface>EffortJointInterface</hardwareInterface>
+       <mechanicalReduction>1</mechanicalReduction>
+     </actuator>
+  </transmission>
+   <link name="l_hip_roll_link">
     <collision>
       <origin xyz="0 0 0" rpy="0 0 0"/>
@@ -347,7 +347,7 @@
     </inertial>
   </link>
-  <joint name="pelvis_yaw_l" type="revolute">
-    <parent link="pelvis_l2"/>
-    <child link="leg_l1"/>
+  <joint name="l_hip_yaw" type="revolute">
+    <parent link="l_hip_roll_link"/>
+    <child link="l_hip_yaw_link"/>
     <origin xyz="0 0 -0.110" rpy="0 0 0"/>
     <axis xyz="0 0 1"/>
@@ -355,15 +355,15 @@
     <dynamics damping = "0.7"/>
   </joint>
-    <transmission name="pelvis_yaw_l_tran">
-     <type>transmission_interface/SimpleTransmission</type>
-     <joint name="pelvis_yaw_l">
-       <hardwareInterface>EffortJointInterface</hardwareInterface>
-     </joint>
-     <actuator name="pelvis_yaw_l_motor">
-       <hardwareInterface>EffortJointInterface</hardwareInterface>
-       <mechanicalReduction>1</mechanicalReduction>
-     </actuator>
-  </transmission>
-   <link name="leg_l1">
+    <transmission name="l_hip_yaw_tran">
+     <type>transmission_interface/SimpleTransmission</type>
+     <joint name="l_hip_yaw">
+       <hardwareInterface>EffortJointInterface</hardwareInterface>
+     </joint>
+     <actuator name="l_hip_yaw">
+       <hardwareInterface>EffortJointInterface</hardwareInterface>
+       <mechanicalReduction>1</mechanicalReduction>
+     </actuator>
+  </transmission>
+   <link name="l_hip_yaw_link">
     <collision>
       <origin xyz="0 0 0" rpy="0 0 0"/>
@@ -385,7 +385,7 @@
     </inertial>
   </link>
-  <joint name="leg_knee_l" type="revolute">
-    <parent link="leg_l1"/>
-    <child link="leg_l2"/>
+  <joint name="l_knee_pitch" type="revolute">
+    <parent link="l_hip_yaw_link"/>
+    <child link="l_knee_pitch_link"/>
     <origin xyz="0 0 -0.170" rpy="0 0 0"/>
     <axis xyz="0 -1 0"/>
@@ -393,15 +393,15 @@
     <dynamics damping = "0.7"/>
   </joint>
-   <transmission name="leg_knee_l_tran">
-     <type>transmission_interface/SimpleTransmission</type>
-     <joint name="leg_knee_l">
-       <hardwareInterface>EffortJointInterface</hardwareInterface>
-     </joint>
-     <actuator name="leg_knee_l_motor">
-       <hardwareInterface>EffortJointInterface</hardwareInterface>
-       <mechanicalReduction>1</mechanicalReduction>
-     </actuator>
-  </transmission>
-   <link name="leg_l2">
+   <transmission name="l_knee_pitch_tran">
+     <type>transmission_interface/SimpleTransmission</type>
+     <joint name="l_knee_pitch">
+       <hardwareInterface>EffortJointInterface</hardwareInterface>
+     </joint>
+     <actuator name="l_knee_pitch_motor">
+       <hardwareInterface>EffortJointInterface</hardwareInterface>
+       <mechanicalReduction>1</mechanicalReduction>
+     </actuator>
+  </transmission>
+   <link name="l_knee_pitch_link">
     <collision>
       <origin xyz="0 0 0" rpy="0 0 0"/>
@@ -423,7 +423,7 @@
     </inertial>
   </link>
-  <joint name="leg_ankle_p_l" type="revolute">
-    <parent link="leg_l2"/>
-    <child link="leg_ankle_l1"/>
+  <joint name="l_ankle_pitch" type="revolute">
+    <parent link="l_knee_pitch_link"/>
+    <child link="l_ankle_pitch_link"/>
     <origin xyz="0 0 -0.28" rpy="0 0 0"/>
     <axis xyz="0 1 0"/>
@@ -431,15 +431,15 @@
     <dynamics damping = "0.7"/>
   </joint>
-  <transmission name="leg_ankle_p_l_tran">
-     <type>transmission_interface/SimpleTransmission</type>
-     <joint name="leg_ankle_p_l">
-       <hardwareInterface>EffortJointInterface</hardwareInterface>
-     </joint>
-     <actuator name="leg_ankle_p_l_motor">
-       <hardwareInterface>EffortJointInterface</hardwareInterface>
-       <mechanicalReduction>1</mechanicalReduction>
-     </actuator>
-  </transmission>
-   <link name="leg_ankle_l1">
+  <transmission name="l_ankle_pitch_tran">
+     <type>transmission_interface/SimpleTransmission</type>
+     <joint name="l_ankle_pitch">
+       <hardwareInterface>EffortJointInterface</hardwareInterface>
+     </joint>
+     <actuator name="l_ankle_pitch_motor">
+       <hardwareInterface>EffortJointInterface</hardwareInterface>
+       <mechanicalReduction>1</mechanicalReduction>
+     </actuator>
+  </transmission>
+   <link name="l_ankle_pitch_link">
     <collision>
       <origin xyz="0 0 0" rpy="0 0 0"/>
@@ -461,7 +461,7 @@
     </inertial>
   </link>
-  <joint name="leg_ankle_r_l" type="revolute">
-    <parent link="leg_ankle_l1"/>
-    <child link="leg_ankle_l2"/>
+  <joint name="l_ankle_roll" type="revolute">
+    <parent link="l_ankle_pitch_link"/>
+    <child link="l_ankle_roll_link"/>
     <origin xyz="0 0 0" rpy="0 0 0"/>
     <axis xyz="1 0 0"/>
@@ -469,15 +469,15 @@
     <dynamics damping = "0.7"/>
   </joint>
-  <transmission name="leg_ankle_r_l_tran">
-     <type>transmission_interface/SimpleTransmission</type>
-     <joint name="leg_ankle_r_l">
-       <hardwareInterface>EffortJointInterface</hardwareInterface>
-     </joint>
-     <actuator name="leg_ankle_r_l_motor">
-       <hardwareInterface>EffortJointInterface</hardwareInterface>
-       <mechanicalReduction>1</mechanicalReduction>
-     </actuator>
-  </transmission>
-   <link name="leg_ankle_l2">
+  <transmission name="l_ankle_roll_tran">
+     <type>transmission_interface/SimpleTransmission</type>
+     <joint name="l_ankle_roll">
+       <hardwareInterface>EffortJointInterface</hardwareInterface>
+     </joint>
+     <actuator name="l_ankle_roll_motor">
+       <hardwareInterface>EffortJointInterface</hardwareInterface>
+       <mechanicalReduction>1</mechanicalReduction>
+     </actuator>
+  </transmission>
+   <link name="l_ankle_roll_link">
     <collision>
       <origin xyz="0 0 0" rpy="0 0 0"/>
@@ -508,7 +508,7 @@
   </link>
 <!-- right -->
-  <joint name="pelvis_pitch_r" type="revolute">
+  <joint name="r_hip_pitch" type="revolute">
     <parent link="pelvis_waist"/>
-    <child link="pelvis_r1"/>
+    <child link="r_hip_pitch_link"/>
     <origin xyz="0 -0.021 0" rpy="0 0 0"/>
     <axis xyz="0 1 0"/>
@@ -516,15 +516,15 @@
     <dynamics damping = "0.7"/>
   </joint>
-    <transmission name="pelvis_pitch_r_tran">
-     <type>transmission_interface/SimpleTransmission</type>
-     <joint name="pelvis_pitch_r">
-       <hardwareInterface>EffortJointInterface</hardwareInterface>
-     </joint>
-     <actuator name="pelvis_pitch_r_motor">
-       <hardwareInterface>EffortJointInterface</hardwareInterface>
-       <mechanicalReduction>1</mechanicalReduction>
-     </actuator>
-  </transmission>
-  <link name="pelvis_r1">
+    <transmission name="r_hip_pitch_tran">
+     <type>transmission_interface/SimpleTransmission</type>
+     <joint name="r_hip_pitch">
+       <hardwareInterface>EffortJointInterface</hardwareInterface>
+     </joint>
+     <actuator name="r_hip_pitch_motor">
+       <hardwareInterface>EffortJointInterface</hardwareInterface>
+       <mechanicalReduction>1</mechanicalReduction>
+     </actuator>
+  </transmission>
+  <link name="r_hip_pitch_link">
     <collision>
       <origin xyz="0 0 0" rpy="0 0 0"/>
@@ -546,7 +546,7 @@
     </inertial>
   </link>
-  <joint name="pelvis_roll_r" type="revolute">
-    <parent link="pelvis_r1"/>
-    <child link="pelvis_r2"/>
+  <joint name="r_hip_roll" type="revolute">
+    <parent link="r_hip_pitch_link"/>
+    <child link="r_hip_roll_link"/>
     <origin xyz="0 -0.059 0" rpy="0 0 0"/>
     <axis xyz="-1 0 0"/>
@@ -554,15 +554,15 @@
     <dynamics damping = "0.7"/>
   </joint>
-  <transmission name="pelvis_roll_r_tran">
-     <type>transmission_interface/SimpleTransmission</type>
-     <joint name="pelvis_roll_r">
-       <hardwareInterface>EffortJointInterface</hardwareInterface>
-     </joint>
-     <actuator name="pelvis_roll_r_motor">
-       <hardwareInterface>EffortJointInterface</hardwareInterface>
-       <mechanicalReduction>1</mechanicalReduction>
-     </actuator>
-  </transmission>
-   <link name="pelvis_r2">
+  <transmission name="r_hip_roll_tran">
+     <type>transmission_interface/SimpleTransmission</type>
+     <joint name="r_hip_roll">
+       <hardwareInterface>EffortJointInterface</hardwareInterface>
+     </joint>
+     <actuator name="r_hip_roll_motor">
+       <hardwareInterface>EffortJointInterface</hardwareInterface>
+       <mechanicalReduction>1</mechanicalReduction>
+     </actuator>
+  </transmission>
+   <link name="r_hip_roll_link">
     <collision>
       <origin xyz="0 0 0" rpy="0 0 0"/>
@@ -584,7 +584,7 @@
     </inertial>
   </link>
-  <joint name="pelvis_yaw_r" type="revolute">
-    <parent link="pelvis_r2"/>
-    <child link="leg_r1"/>
+  <joint name="r_hip_yaw" type="revolute">
+    <parent link="r_hip_roll_link"/>
+    <child link="r_hip_yaw_link"/>
     <origin xyz="0 0 -0.110" rpy="0 0 0"/>
     <axis xyz="0 0 1"/>
@@ -592,15 +592,15 @@
     <dynamics damping = "0.7"/>
   </joint>
-  <transmission name="pelvis_yaw_r_tran">
-     <type>transmission_interface/SimpleTransmission</type>
-     <joint name="pelvis_yaw_r">
-       <hardwareInterface>EffortJointInterface</hardwareInterface>
-     </joint>
-     <actuator name="pelvis_yaw_r_motor">
-       <hardwareInterface>EffortJointInterface</hardwareInterface>
-       <mechanicalReduction>1</mechanicalReduction>
-     </actuator>
-  </transmission>
-   <link name="leg_r1">
+  <transmission name="r_hip_yaw_tran">
+     <type>transmission_interface/SimpleTransmission</type>
+     <joint name="r_hip_yaw">
+       <hardwareInterface>EffortJointInterface</hardwareInterface>
+     </joint>
+     <actuator name="r_hip_yaw_motor">
+       <hardwareInterface>EffortJointInterface</hardwareInterface>
+       <mechanicalReduction>1</mechanicalReduction>
+     </actuator>
+  </transmission>
+   <link name="r_hip_yaw_link">
     <collision>
       <origin xyz="0 0 0" rpy="0 0 0"/>
@@ -622,7 +622,7 @@
     </inertial>
   </link>
-  <joint name="leg_knee_r" type="revolute">
-    <parent link="leg_r1"/>
-    <child link="leg_r2"/>
+  <joint name="r_knee_pitch" type="revolute">
+    <parent link="r_hip_yaw_link"/>
+    <child link="r_knee_pitch_link"/>
     <origin xyz="0 0 -0.17" rpy="0 0 0"/>
     <axis xyz="0 1 0"/>
@@ -630,15 +630,15 @@
     <dynamics damping = "0.7"/>
   </joint>
-   <transmission name="leg_knee_r_tran">
-     <type>transmission_interface/SimpleTransmission</type>
-     <joint name="leg_knee_r">
-       <hardwareInterface>EffortJointInterface</hardwareInterface>
-     </joint>
-     <actuator name="leg_knee_r_motor">
-       <hardwareInterface>EffortJointInterface</hardwareInterface>
-       <mechanicalReduction>1</mechanicalReduction>
-     </actuator>
-  </transmission>
-   <link name="leg_r2">
+   <transmission name="r_knee_pitch_tran">
+     <type>transmission_interface/SimpleTransmission</type>
+     <joint name="r_knee_pitch">
+       <hardwareInterface>EffortJointInterface</hardwareInterface>
+     </joint>
+     <actuator name="r_knee_pitch_motor">
+       <hardwareInterface>EffortJointInterface</hardwareInterface>
+       <mechanicalReduction>1</mechanicalReduction>
+     </actuator>
+  </transmission>
+   <link name="r_knee_pitch_link">
     <collision>
       <origin xyz="0 0 0" rpy="0 0 0"/>
@@ -660,7 +660,7 @@
     </inertial>
   </link>
-  <joint name="leg_ankle_p_r" type="revolute">
-    <parent link="leg_r2"/>
-    <child link="leg_ankle_r1"/>
+  <joint name="r_ankle_pitch" type="revolute">
+    <parent link="r_knee_pitch_link"/>
+    <child link="r_ankle_pitch_link"/>
     <origin xyz="0 0 -0.28" rpy="0 0 0"/>
     <axis xyz="0 -1 0"/>
@@ -668,15 +668,15 @@
     <dynamics damping = "0.7"/>
   </joint>
-  <transmission name="leg_ankle_p_r_tran">
-     <type>transmission_interface/SimpleTransmission</type>
-     <joint name="leg_ankle_p_r">
-       <hardwareInterface>EffortJointInterface</hardwareInterface>
-     </joint>
-     <actuator name="leg_ankle_p_r_motor">
-       <hardwareInterface>EffortJointInterface</hardwareInterface>
-       <mechanicalReduction>1</mechanicalReduction>
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