Commit message: model_modified

File: alice_2_description/urdf/alice_2_robot.xacro (robot description, xacro)
@@ -114,7 +114,7 @@
   </link>
 <!-- left_leg -->
-  <joint name="pelvis_pitch_l" type="revolute">
+  <joint name="l_hip_pitch" type="revolute">
     <parent link="pelvis_waist"/>
-    <child link="pelvis_l1"/>
+    <child link="l_hip_pitch_link"/>
     <origin xyz="0 0 0" rpy="0 0 0"/>
     <axis xyz="0 -1 0"/>
@@ -122,15 +122,15 @@
     <dynamics damping = "0.7"/>
   </joint>
-  <transmission name="pelvis_pitch_l_tran">
-     <type>transmission_interface/SimpleTransmission</type>
-     <joint name="pelvis_pitch_l">
-       <hardwareInterface>EffortJointInterface</hardwareInterface>
-     </joint>
-     <actuator name="pelvis_pitch_l_motor">
-       <hardwareInterface>EffortJointInterface</hardwareInterface>
-       <mechanicalReduction>1</mechanicalReduction>
-     </actuator>
-  </transmission>
-  <link name="pelvis_l1">
+  <transmission name="l_hip_pitch_tran">
+     <type>transmission_interface/SimpleTransmission</type>
+     <joint name="l_hip_pitch">
+       <hardwareInterface>EffortJointInterface</hardwareInterface>
+     </joint>
+     <actuator name="l_hip_pitch_motor">
+       <hardwareInterface>EffortJointInterface</hardwareInterface>
+       <mechanicalReduction>1</mechanicalReduction>
+     </actuator>
+  </transmission>
+  <link name="l_hip_pitch_link">
     <collision>
       <origin xyz="0 0 0" rpy="0 0 0"/>
@@ -152,7 +152,7 @@
     </inertial>
   </link>
-  <joint name="pelvis_roll_l" type="revolute">
-    <parent link="pelvis_l1"/>
-    <child link="pelvis_l2"/>
+  <joint name="l_hip_roll" type="revolute">
+    <parent link="l_hip_pitch_link"/>
+    <child link="l_hip_roll_link"/>
     <origin xyz="0 0.09 0" rpy="0 0 0"/>
     <axis xyz="-1 0 0"/>
@@ -160,15 +160,15 @@
     <dynamics damping = "0.7"/>
   </joint>
-  <transmission name="pelvis_roll_l_tran">
-     <type>transmission_interface/SimpleTransmission</type>
-     <joint name="pelvis_roll_l">
-       <hardwareInterface>EffortJointInterface</hardwareInterface>
-     </joint>
-     <actuator name="pelvis_roll_l_motor">
-       <hardwareInterface>EffortJointInterface</hardwareInterface>
-       <mechanicalReduction>1</mechanicalReduction>
-     </actuator>
-  </transmission>
-   <link name="pelvis_l2">
+  <transmission name="l_hip_roll_tran">
+     <type>transmission_interface/SimpleTransmission</type>
+     <joint name="l_hip_roll">
+       <hardwareInterface>EffortJointInterface</hardwareInterface>
+     </joint>
+     <actuator name="l_hip_roll_motor">
+       <hardwareInterface>EffortJointInterface</hardwareInterface>
+       <mechanicalReduction>1</mechanicalReduction>
+     </actuator>
+  </transmission>
+   <link name="l_hip_roll_link">
     <collision>
       <origin xyz="0 0 0" rpy="0 0 0"/>
@@ -190,7 +190,7 @@
     </inertial>
   </link>
-  <joint name="pelvis_yaw_l" type="revolute">
-    <parent link="pelvis_l2"/>
-    <child link="leg_l1"/>
+  <joint name="l_hip_yaw" type="revolute">
+    <parent link="l_hip_roll_link"/>
+    <child link="l_hip_yaw_link"/>
     <origin xyz="0 0 -0.133875" rpy="0 0 0"/>
     <axis xyz="0 0 1"/>
@@ -198,15 +198,15 @@
     <dynamics damping = "0.7"/>
   </joint>
-    <transmission name="pelvis_yaw_l_tran">
-     <type>transmission_interface/SimpleTransmission</type>
-     <joint name="pelvis_yaw_l">
-       <hardwareInterface>EffortJointInterface</hardwareInterface>
-     </joint>
-     <actuator name="pelvis_yaw_l_motor">
-       <hardwareInterface>EffortJointInterface</hardwareInterface>
-       <mechanicalReduction>1</mechanicalReduction>
-     </actuator>
-  </transmission>
-   <link name="leg_l1">
+    <transmission name="l_hip_yaw_tran">
+     <type>transmission_interface/SimpleTransmission</type>
+     <joint name="l_hip_yaw">
+       <hardwareInterface>EffortJointInterface</hardwareInterface>
+     </joint>
+     <actuator name="l_hip_yaw_motor">
+       <hardwareInterface>EffortJointInterface</hardwareInterface>
+       <mechanicalReduction>1</mechanicalReduction>
+     </actuator>
+  </transmission>
+   <link name="l_hip_yaw_link">
     <collision>
       <origin xyz="0 0 0" rpy="0 0 0"/>
@@ -228,7 +228,7 @@
     </inertial>
   </link>
-  <joint name="leg_knee_l" type="revolute">
-    <parent link="leg_l1"/>
-    <child link="leg_l2"/>
+  <joint name="l_knee_pitch" type="revolute">
+    <parent link="l_hip_yaw_link"/>
+    <child link="l_knee_pitch_link"/>
     <origin xyz="0 0 -0.106125" rpy="0 0 0"/>
     <axis xyz="0 -1 0"/>
@@ -236,15 +236,15 @@
     <dynamics damping = "0.7"/>
   </joint>
-   <transmission name="leg_knee_l_tran">
-     <type>transmission_interface/SimpleTransmission</type>
-     <joint name="leg_knee_l">
-       <hardwareInterface>EffortJointInterface</hardwareInterface>
-     </joint>
-     <actuator name="leg_knee_l_motor">
-       <hardwareInterface>EffortJointInterface</hardwareInterface>
-       <mechanicalReduction>1</mechanicalReduction>
-     </actuator>
-  </transmission>
-   <link name="leg_l2">
+   <transmission name="l_knee_pitch_tran">
+     <type>transmission_interface/SimpleTransmission</type>
+     <joint name="l_knee_pitch">
+       <hardwareInterface>EffortJointInterface</hardwareInterface>
+     </joint>
+     <actuator name="l_knee_pitch_motor">
+       <hardwareInterface>EffortJointInterface</hardwareInterface>
+       <mechanicalReduction>1</mechanicalReduction>
+     </actuator>
+  </transmission>
+   <link name="l_knee_pitch_link">
     <collision>
       <origin xyz="0 0 0" rpy="0 0 0"/>
@@ -266,7 +266,7 @@
     </inertial>
   </link>
-  <joint name="leg_ankle_p_l" type="revolute">
-    <parent link="leg_l2"/>
-    <child link="leg_ankle_l1"/>
+  <joint name="l_ankle_pitch" type="revolute">
+    <parent link="l_knee_pitch_link"/>
+    <child link="l_ankle_pitch_link"/>
     <origin xyz="0 0 -0.24" rpy="0 0 0"/>
     <axis xyz="0 1 0"/>
@@ -274,15 +274,15 @@
     <dynamics damping = "0.7"/>
   </joint>
-  <transmission name="leg_ankle_p_l_tran">
-     <type>transmission_interface/SimpleTransmission</type>
-     <joint name="leg_ankle_p_l">
-       <hardwareInterface>EffortJointInterface</hardwareInterface>
-     </joint>
-     <actuator name="leg_ankle_p_l_motor">
-       <hardwareInterface>EffortJointInterface</hardwareInterface>
-       <mechanicalReduction>1</mechanicalReduction>
-     </actuator>
-  </transmission>
-   <link name="leg_ankle_l1">
+  <transmission name="l_ankle_pitch_tran">
+     <type>transmission_interface/SimpleTransmission</type>
+     <joint name="l_ankle_pitch">
+       <hardwareInterface>EffortJointInterface</hardwareInterface>
+     </joint>
+     <actuator name="l_ankle_pitch_motor">
+       <hardwareInterface>EffortJointInterface</hardwareInterface>
+       <mechanicalReduction>1</mechanicalReduction>
+     </actuator>
+  </transmission>
+   <link name="l_ankle_pitch_link">
     <collision>
       <origin xyz="0 0 0" rpy="0 0 0"/>
@@ -304,7 +304,7 @@
     </inertial>
   </link>
-  <joint name="leg_ankle_r_l" type="revolute">
-    <parent link="leg_ankle_l1"/>
-    <child link="leg_ankle_l2"/>
+  <joint name="l_ankle_roll" type="revolute">
+    <parent link="l_ankle_pitch_link"/>
+    <child link="l_ankle_roll_link"/>
     <origin xyz="0 0 0" rpy="0 0 0"/>
     <axis xyz="1 0 0"/>
@@ -312,15 +312,15 @@
     <dynamics damping = "0.7"/>
   </joint>
-  <transmission name="leg_ankle_r_l_tran">
-     <type>transmission_interface/SimpleTransmission</type>
-     <joint name="leg_ankle_r_l">
-       <hardwareInterface>EffortJointInterface</hardwareInterface>
-     </joint>
-     <actuator name="leg_ankle_r_l_motor">
-       <hardwareInterface>EffortJointInterface</hardwareInterface>
-       <mechanicalReduction>1</mechanicalReduction>
-     </actuator>
-  </transmission>
-   <link name="leg_ankle_l2">
+  <transmission name="l_ankle_roll_tran">
+     <type>transmission_interface/SimpleTransmission</type>
+     <joint name="l_ankle_roll">
+       <hardwareInterface>EffortJointInterface</hardwareInterface>
+     </joint>
+     <actuator name="l_ankle_roll_motor">
+       <hardwareInterface>EffortJointInterface</hardwareInterface>
+       <mechanicalReduction>1</mechanicalReduction>
+     </actuator>
+  </transmission>
+   <link name="l_ankle_roll_link">
     <collision>
       <origin xyz="0 0 0" rpy="0 0 0"/>
@@ -343,7 +343,7 @@
   </link>
 <!-- right -->
-  <joint name="pelvis_pitch_r" type="revolute">
+  <joint name="r_hip_pitch" type="revolute">
     <parent link="pelvis_waist"/>
-    <child link="pelvis_r1"/>
+    <child link="r_hip_pitch_link"/>
     <origin xyz="0 0 0" rpy="0 0 0"/>
     <axis xyz="0 1 0"/>
@@ -351,15 +351,15 @@
     <dynamics damping = "0.7"/>
   </joint>
-    <transmission name="pelvis_pitch_r_tran">
-     <type>transmission_interface/SimpleTransmission</type>
-     <joint name="pelvis_pitch_r">
-       <hardwareInterface>EffortJointInterface</hardwareInterface>
-     </joint>
-     <actuator name="pelvis_pitch_r_motor">
-       <hardwareInterface>EffortJointInterface</hardwareInterface>
-       <mechanicalReduction>1</mechanicalReduction>
-     </actuator>
-  </transmission>
-  <link name="pelvis_r1">
+    <transmission name="r_hip_pitch_tran">
+     <type>transmission_interface/SimpleTransmission</type>
+     <joint name="r_hip_pitch">
+       <hardwareInterface>EffortJointInterface</hardwareInterface>
+     </joint>
+     <actuator name="r_hip_pitch_motor">
+       <hardwareInterface>EffortJointInterface</hardwareInterface>
+       <mechanicalReduction>1</mechanicalReduction>
+     </actuator>
+  </transmission>
+  <link name="r_hip_pitch_link">
     <collision>
       <origin xyz="0 0 0" rpy="0 0 0"/>
@@ -381,7 +381,7 @@
     </inertial>
   </link>
-  <joint name="pelvis_roll_r" type="revolute">
-    <parent link="pelvis_r1"/>
-    <child link="pelvis_r2"/>
+  <joint name="r_hip_roll" type="revolute">
+    <parent link="r_hip_pitch_link"/>
+    <child link="r_hip_roll_link"/>
     <origin xyz="0 -0.09 0" rpy="0 0 0"/>
     <axis xyz="-1 0 0"/>
@@ -389,15 +389,15 @@
     <dynamics damping = "0.7"/>
   </joint>
-  <transmission name="pelvis_roll_r_tran">
-     <type>transmission_interface/SimpleTransmission</type>
-     <joint name="pelvis_roll_r">
-       <hardwareInterface>EffortJointInterface</hardwareInterface>
-     </joint>
-     <actuator name="pelvis_roll_r_motor">
-       <hardwareInterface>EffortJointInterface</hardwareInterface>
-       <mechanicalReduction>1</mechanicalReduction>
-     </actuator>
-  </transmission>
-   <link name="pelvis_r2">
+  <transmission name="r_hip_roll_tran">
+     <type>transmission_interface/SimpleTransmission</type>
+     <joint name="r_hip_roll">
+       <hardwareInterface>EffortJointInterface</hardwareInterface>
+     </joint>
+     <actuator name="r_hip_roll_motor">
+       <hardwareInterface>EffortJointInterface</hardwareInterface>
+       <mechanicalReduction>1</mechanicalReduction>
+     </actuator>
+  </transmission>
+   <link name="r_hip_roll_link">
     <collision>
       <origin xyz="0 0 0" rpy="0 0 0"/>
@@ -419,7 +419,7 @@
     </inertial>
   </link>
-  <joint name="pelvis_yaw_r" type="revolute">
-    <parent link="pelvis_r2"/>
-    <child link="leg_r1"/>
+  <joint name="r_hip_yaw" type="revolute">
+    <parent link="r_hip_roll_link"/>
+    <child link="r_hip_yaw_link"/>
     <origin xyz="0 0 -0.133875" rpy="0 0 0"/>
     <axis xyz="0 0 1"/>
@@ -427,15 +427,15 @@
     <dynamics damping = "0.7"/>
   </joint>
-  <transmission name="pelvis_yaw_r_tran">
-     <type>transmission_interface/SimpleTransmission</type>
-     <joint name="pelvis_yaw_r">
-       <hardwareInterface>EffortJointInterface</hardwareInterface>
-     </joint>
-     <actuator name="pelvis_yaw_r_motor">
-       <hardwareInterface>EffortJointInterface</hardwareInterface>
-       <mechanicalReduction>1</mechanicalReduction>
-     </actuator>
-  </transmission>
-   <link name="leg_r1">
+  <transmission name="r_hip_yaw_tran">
+     <type>transmission_interface/SimpleTransmission</type>
+     <joint name="r_hip_yaw">
+       <hardwareInterface>EffortJointInterface</hardwareInterface>
+     </joint>
+     <actuator name="r_hip_yaw_motor">
+       <hardwareInterface>EffortJointInterface</hardwareInterface>
+       <mechanicalReduction>1</mechanicalReduction>
+     </actuator>
+  </transmission>
+   <link name="r_hip_yaw_link">
     <collision>
       <origin xyz="0 0 0" rpy="0 0 0"/>
@@ -457,7 +457,7 @@
     </inertial>
   </link>
-  <joint name="leg_knee_r" type="revolute">
-    <parent link="leg_r1"/>
-    <child link="leg_r2"/>
+  <joint name="r_knee_pitch" type="revolute">
+    <parent link="r_hip_yaw_link"/>
+    <child link="r_knee_pitch_link"/>
     <origin xyz="0 0 -0.106125" rpy="0 0 0"/>
     <axis xyz="0 1 0"/>
@@ -465,15 +465,15 @@
     <dynamics damping = "0.7"/>
   </joint>
-   <transmission name="leg_knee_r_tran">
-     <type>transmission_interface/SimpleTransmission</type>
-     <joint name="leg_knee_r">
-       <hardwareInterface>EffortJointInterface</hardwareInterface>
-     </joint>
-     <actuator name="leg_knee_r_motor">
-       <hardwareInterface>EffortJointInterface</hardwareInterface>
-       <mechanicalReduction>1</mechanicalReduction>
-     </actuator>
-  </transmission>
-   <link name="leg_r2">
+   <transmission name="r_knee_pitch_tran">
+     <type>transmission_interface/SimpleTransmission</type>
+     <joint name="r_knee_pitch">
+       <hardwareInterface>EffortJointInterface</hardwareInterface>
+     </joint>
+     <actuator name="r_knee_pitch_motor">
+       <hardwareInterface>EffortJointInterface</hardwareInterface>
+       <mechanicalReduction>1</mechanicalReduction>
+     </actuator>
+  </transmission>
+   <link name="r_knee_pitch_link">
     <collision>
       <origin xyz="0 0 0" rpy="0 0 0"/>
@@ -495,7 +495,7 @@
     </inertial>
   </link>
-  <joint name="leg_ankle_p_r" type="revolute">
-    <parent link="leg_r2"/>
-    <child link="leg_ankle_r1"/>
+  <joint name="r_ankle_pitch" type="revolute">
+    <parent link="r_knee_pitch_link"/>
+    <child link="r_ankle_pitch_link"/>
     <origin xyz="0 0 -0.24" rpy="0 0 0"/>
     <axis xyz="0 -1 0"/>
@@ -503,15 +503,15 @@
     <dynamics damping = "0.7"/>
   </joint>
-  <transmission name="leg_ankle_p_r_tran">
-     <type>transmission_interface/SimpleTransmission</type>
-     <joint name="leg_ankle_p_r">
-       <hardwareInterface>EffortJointInterface</hardwareInterface>
-     </joint>
-     <actuator name="leg_ankle_p_r_motor">
-       <hardwareInterface>EffortJointInterface</hardwareInterface>
-       <mechanicalReduction>1</mechanicalReduction>
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
Commit message: m

File: alice_1_description/urdf/alice_1_robot.xacro (robot description, xacro)
@@ -78,5 +78,5 @@
     <parent link="pelvis_waist"/>
     <child link="head_yaw_link"/>
-    <origin xyz="0 0 0.4665" rpy="0 0 0"/>
+    <origin xyz="0 0 0.4435" rpy="0 0 0"/>
     <axis xyz="0 0 1"/>
     <limit velocity="6.5" effort="1000" lower="${-pi/2}" upper="${pi}" />
@@ -116,5 +116,5 @@
     <parent link="head_yaw_link"/>
     <child link="head_pitch_link"/>
-    <origin xyz="0 0 0" rpy="0 0 0"/>
+    <origin xyz="0 0 0.023" rpy="0 0 0"/>
     <axis xyz="0 1 0"/>
     <limit velocity="6.5" effort="1000" lower="${-pi/2}" upper="${pi}" />
@@ -135,11 +135,11 @@
       <origin xyz="0 0 0" rpy="0 0 0"/>
       <geometry>
-          <mesh filename="package://alice_1_description/meshes/asm_hum_fb_3_head_y1.stl" scale="0.001 0.001 0.001"/>
-        </geometry>
-    </collision>
-    <visual>
-        <origin xyz="0 0 0" rpy="0 0 0"/>
-        <geometry>
-          <mesh filename="package://alice_1_description/meshes/asm_hum_fb_3_head_y1.stl" scale="0.001 0.001 0.001"/>
+          <mesh filename="package://alice_1_description/meshes/asm_hum_fb_3_head_p1.stl" scale="0.001 0.001 0.001"/>
+        </geometry>
+    </collision>
+    <visual>
+        <origin xyz="0 0 0" rpy="0 0 0"/>
+        <geometry>
+          <mesh filename="package://alice_1_description/meshes/asm_hum_fb_3_head_p1.stl" scale="0.001 0.001 0.001"/>
         </geometry>
         <material name="red"/>
@@ -155,5 +155,5 @@
     <parent link="head_pitch_link"/>
     <child link="head_fake_link"/>
-    <origin xyz="0 0 0.13" rpy="0 0 0"/>
+    <origin xyz="0 0 0.16" rpy="0 0 0"/>
     <axis xyz="0 1 0"/>
     <limit velocity="6.5" effort="1000" lower="${-pi/2}" upper="${pi}" />
