Commit message: modified

File: alice_1_description/urdf/alice_1_robot.xacro (robot description, xacro)
@@ -192,4 +192,5 @@
     </inertial>
   </link>
+<!-- left arm -->
 <!-- l_shoulder_pitch -->
   <joint name="l_shoulder_pitch" type="revolute">
@@ -231,4 +232,81 @@
     </inertial>
   </link>
+  <joint name="l_shoulder_roll" type="revolute">
+    <parent link="l_shoulder_pitch_link"/>
+    <child link="l_shoulder_roll_link"/>
+    <origin xyz="0 0 0" rpy="0 0 0"/>
+    <axis xyz="1 0 0"/>
+    <limit velocity="6.5" effort="1000" lower="${-pi/2}" upper="${pi}" />
+    <dynamics damping = "0.7"/>
+  </joint>
+  <transmission name="l_shoulder_roll_tran">
+     <type>transmission_interface/SimpleTransmission</type>
+     <joint name="l_shoulder_roll">
+       <hardwareInterface>EffortJointInterface</hardwareInterface>
+     </joint>
+     <actuator name="l_shoulder_roll_motor">
+       <hardwareInterface>EffortJointInterface</hardwareInterface>
+       <mechanicalReduction>1</mechanicalReduction>
+     </actuator>
+  </transmission>
+  <link name="l_shoulder_roll_link">
+    <collision>
+      <origin xyz="0 0 0" rpy="0 0 0"/>
+      <geometry>
+          <mesh filename="package://alice_1_description/meshes/prt_hum_fb_3_elbow_l.stl" scale="0.001 0.001 0.001"/>
+        </geometry>
+    </collision>
+    <visual>
+        <origin xyz="0 0 0" rpy="0 0 0"/>
+        <geometry>
+          <mesh filename="package://alice_1_description/meshes/prt_hum_fb_3_elbow_l.stl" scale="0.001 0.001 0.001"/>
+        </geometry>
+        <material name="red"/>
+    </visual>
+    <inertial>
+      <origin xyz="0 0 0" rpy="0 0 0"/>
+      <mass value="1"/>
+      <inertia ixx="1.0" ixy="0.0" ixz="0.0" iyy="1.0" iyz="0.0" izz="1.0" />
+    </inertial>
+  </link>
+ <joint name="l_elbow_pitch" type="revolute">
+    <parent link="l_shoulder_roll_link"/>
+    <child link="l_elbow_pitch_link"/>
+    <origin xyz="0 0 -0.27" rpy="0 0 0"/>
+    <axis xyz="0 1 0"/>
+    <limit velocity="6.5" effort="1000" lower="${-pi/2}" upper="${pi}" />
+    <dynamics damping = "0.7"/>
+  </joint>
+  <transmission name="l_elbow_pitch_tran">
+     <type>transmission_interface/SimpleTransmission</type>
+     <joint name="l_elbow_pitch">
+       <hardwareInterface>EffortJointInterface</hardwareInterface>
+     </joint>
+     <actuator name="l_elbow_pitch_motor">
+       <hardwareInterface>EffortJointInterface</hardwareInterface>
+       <mechanicalReduction>1</mechanicalReduction>
+     </actuator>
+  </transmission>
+  <link name="l_elbow_pitch_link">
+    <collision>
+      <origin xyz="0 0 0" rpy="0 0 0"/>
+      <geometry>
+          <mesh filename="package://alice_1_description/meshes/prt_hum_fb_3_elbo_2_l.stl" scale="0.001 0.001 0.001"/>
+        </geometry>
+    </collision>
+    <visual>
+        <origin xyz="0 0 0" rpy="0 0 0"/>
+        <geometry>
+          <mesh filename="package://alice_1_description/meshes/prt_hum_fb_3_elbo_2_l.stl" scale="0.001 0.001 0.001"/>
+        </geometry>
+        <material name="red"/>
+    </visual>
+    <inertial>
+      <origin xyz="0 0 0" rpy="0 0 0"/>
+      <mass value="1"/>
+      <inertia ixx="1.0" ixy="0.0" ixz="0.0" iyy="1.0" iyz="0.0" izz="1.0" />
+    </inertial>
+  </link>
+<!-- right arm -->
 <!-- r_shoulder_pitch -->
  <joint name="r_shoulder_pitch" type="revolute">
@@ -261,4 +339,80 @@
         <geometry>
           <mesh filename="package://alice_1_description/meshes/asm_hum_fb_3_shr_r1.stl" scale="0.001 0.001 0.001"/>
+        </geometry>
+        <material name="red"/>
+    </visual>
+    <inertial>
+      <origin xyz="0 0 0" rpy="0 0 0"/>
+      <mass value="1"/>
+      <inertia ixx="1.0" ixy="0.0" ixz="0.0" iyy="1.0" iyz="0.0" izz="1.0" />
+    </inertial>
+  </link>
+ <joint name="r_shoulder_roll" type="revolute">
+    <parent link="r_shoulder_pitch_link"/>
+    <child link="r_shoulder_roll_link"/>
+    <origin xyz="0 0 0" rpy="0 0 0"/>
+    <axis xyz="1 0 0"/>
+    <limit velocity="6.5" effort="1000" lower="${-pi/2}" upper="${pi}" />
+    <dynamics damping = "0.7"/>
+  </joint>
+  <transmission name="r_shoulder_roll_tran">
+     <type>transmission_interface/SimpleTransmission</type>
+     <joint name="r_shoulder_roll">
+       <hardwareInterface>EffortJointInterface</hardwareInterface>
+     </joint>
+     <actuator name="r_shoulder_roll_motor">
+       <hardwareInterface>EffortJointInterface</hardwareInterface>
+       <mechanicalReduction>1</mechanicalReduction>
+     </actuator>
+  </transmission>
+  <link name="r_shoulder_roll_link">
+    <collision>
+      <origin xyz="0 0 0" rpy="0 0 0"/>
+      <geometry>
+          <mesh filename="package://alice_1_description/meshes/prt_hum_fb_3_elbow_l.stl" scale="0.001 0.001 0.001"/>
+        </geometry>
+    </collision>
+    <visual>
+        <origin xyz="0 0 0" rpy="0 0 0"/>
+        <geometry>
+          <mesh filename="package://alice_1_description/meshes/prt_hum_fb_3_elbow_l.stl" scale="0.001 0.001 0.001"/>
+        </geometry>
+        <material name="red"/>
+    </visual>
+    <inertial>
+      <origin xyz="0 0 0" rpy="0 0 0"/>
+      <mass value="1"/>
+      <inertia ixx="1.0" ixy="0.0" ixz="0.0" iyy="1.0" iyz="0.0" izz="1.0" />
+    </inertial>
+  </link>
+ <joint name="r_elbow_pitch" type="revolute">
+    <parent link="r_shoulder_roll_link"/>
+    <child link="r_elbow_pitch_link"/>
+    <origin xyz="0 0 -0.27" rpy="0 0 0"/>
+    <axis xyz="0 -1 0"/>
+    <limit velocity="6.5" effort="1000" lower="${-pi/2}" upper="${pi}" />
+    <dynamics damping = "0.7"/>
+  </joint>
+  <transmission name="r_elbow_pitch_tran">
+     <type>transmission_interface/SimpleTransmission</type>
+     <joint name="r_elbow_pitch">
+       <hardwareInterface>EffortJointInterface</hardwareInterface>
+     </joint>
+     <actuator name="r_elbow_pitch_motor">
+       <hardwareInterface>EffortJointInterface</hardwareInterface>
+       <mechanicalReduction>1</mechanicalReduction>
+     </actuator>
+  </transmission>
+  <link name="r_elbow_pitch_link">
+    <collision>
+      <origin xyz="0 0 0" rpy="0 0 0"/>
+      <geometry>
+          <mesh filename="package://alice_1_description/meshes/prt_hum_fb_3_elbo_2_l.stl" scale="0.001 0.001 0.001"/>
+        </geometry>
+    </collision>
+    <visual>
+        <origin xyz="0 0 0" rpy="0 0 0"/>
+        <geometry>
+          <mesh filename="package://alice_1_description/meshes/prt_hum_fb_3_elbo_2_l.stl" scale="0.001 0.001 0.001"/>
         </geometry>
         <material name="red"/>

File: alice_2_description/urdf/alice_2_robot.xacro (robot description, xacro)
@@ -72,4 +72,236 @@
     </inertial>
   </link>
+<!-- left arm -->
+<!-- l_shoulder_pitch -->
+  <joint name="l_shoulder_pitch" type="revolute">
+    <parent link="chest_fixed"/>
+    <child link="l_shoulder_pitch_link"/>
+    <origin xyz="0 0.175 0.08" rpy="0 0 0"/>
+    <axis xyz="0 1 0"/>
+    <limit velocity="6.5" effort="1000" lower="${-pi/2}" upper="${pi}" />
+    <dynamics damping = "0.7"/>
+  </joint>
+  <transmission name="l_shoulder_pitch_tran">
+     <type>transmission_interface/SimpleTransmission</type>
+     <joint name="l_shoulder_pitch">
+       <hardwareInterface>EffortJointInterface</hardwareInterface>
+     </joint>
+     <actuator name="l_shoulder_pitch_motor">
+       <hardwareInterface>EffortJointInterface</hardwareInterface>
+       <mechanicalReduction>1</mechanicalReduction>
+     </actuator>
+  </transmission>
+  <link name="l_shoulder_pitch_link">
+    <collision>
+      <origin xyz="0 0 0" rpy="0 0 0"/>
+      <geometry>
+          <mesh filename="package://alice_1_description/meshes/asm_hum_fb_3_shr_l1.stl" scale="0.001 0.001 0.001"/>
+        </geometry>
+    </collision>
+    <visual>
+        <origin xyz="0 0 0" rpy="0 0 0"/>
+        <geometry>
+          <mesh filename="package://alice_1_description/meshes/asm_hum_fb_3_shr_l1.stl" scale="0.001 0.001 0.001"/>
+        </geometry>
+        <material name="red"/>
+    </visual>
+    <inertial>
+      <origin xyz="0 0 0" rpy="0 0 0"/>
+      <mass value="1"/>
+      <inertia ixx="1.0" ixy="0.0" ixz="0.0" iyy="1.0" iyz="0.0" izz="1.0" />
+    </inertial>
+  </link>
+  <joint name="l_shoulder_roll" type="revolute">
+    <parent link="l_shoulder_pitch_link"/>
+    <child link="l_shoulder_roll_link"/>
+    <origin xyz="0 0 0" rpy="0 0 0"/>
+    <axis xyz="1 0 0"/>
+    <limit velocity="6.5" effort="1000" lower="${-pi/2}" upper="${pi}" />
+    <dynamics damping = "0.7"/>
+  </joint>
+  <transmission name="l_shoulder_roll_tran">
+     <type>transmission_interface/SimpleTransmission</type>
+     <joint name="l_shoulder_roll">
+       <hardwareInterface>EffortJointInterface</hardwareInterface>
+     </joint>
+     <actuator name="l_shoulder_roll_motor">
+       <hardwareInterface>EffortJointInterface</hardwareInterface>
+       <mechanicalReduction>1</mechanicalReduction>
+     </actuator>
+  </transmission>
+  <link name="l_shoulder_roll_link">
+    <collision>
+      <origin xyz="0 0 0" rpy="0 0 0"/>
+      <geometry>
+          <mesh filename="package://alice_1_description/meshes/prt_hum_fb_3_elbow_l.stl" scale="0.001 0.001 0.001"/>
+        </geometry>
+    </collision>
+    <visual>
+        <origin xyz="0 0 0" rpy="0 0 0"/>
+        <geometry>
+          <mesh filename="package://alice_1_description/meshes/prt_hum_fb_3_elbow_l.stl" scale="0.001 0.001 0.001"/>
+        </geometry>
+        <material name="red"/>
+    </visual>
+    <inertial>
+      <origin xyz="0 0 0" rpy="0 0 0"/>
+      <mass value="1"/>
+      <inertia ixx="1.0" ixy="0.0" ixz="0.0" iyy="1.0" iyz="0.0" izz="1.0" />
+    </inertial>
+  </link>
+ <joint name="l_elbow_pitch" type="revolute">
+    <parent link="l_shoulder_roll_link"/>
+    <child link="l_elbow_pitch_link"/>
+    <origin xyz="0 0 -0.27" rpy="0 0 0"/>
+    <axis xyz="0 1 0"/>
+    <limit velocity="6.5" effort="1000" lower="${-pi/2}" upper="${pi}" />
+    <dynamics damping = "0.7"/>
+  </joint>
+  <transmission name="l_elbow_pitch_tran">
+     <type>transmission_interface/SimpleTransmission</type>
+     <joint name="l_elbow_pitch">
+       <hardwareInterface>EffortJointInterface</hardwareInterface>
+     </joint>
+     <actuator name="l_elbow_pitch_motor">
+       <hardwareInterface>EffortJointInterface</hardwareInterface>
+       <mechanicalReduction>1</mechanicalReduction>
+     </actuator>
+  </transmission>
+  <link name="l_elbow_pitch_link">
+    <collision>
+      <origin xyz="0 0 0" rpy="0 0 0"/>
+      <geometry>
+          <mesh filename="package://alice_1_description/meshes/prt_hum_fb_3_elbo_2_l.stl" scale="0.001 0.001 0.001"/>
+        </geometry>
+    </collision>
+    <visual>
+        <origin xyz="0 0 0" rpy="0 0 0"/>
+        <geometry>
+          <mesh filename="package://alice_1_description/meshes/prt_hum_fb_3_elbo_2_l.stl" scale="0.001 0.001 0.001"/>
+        </geometry>
+        <material name="red"/>
+    </visual>
+    <inertial>
+      <origin xyz="0 0 0" rpy="0 0 0"/>
+      <mass value="1"/>
+      <inertia ixx="1.0" ixy="0.0" ixz="0.0" iyy="1.0" iyz="0.0" izz="1.0" />
+    </inertial>
+  </link>
+<!-- right arm -->
+<!-- r_shoulder_pitch -->
+ <joint name="r_shoulder_pitch" type="revolute">
+    <parent link="chest_fixed"/>
+    <child link="r_shoulder_pitch_link"/>
+    <origin xyz="0 -0.175 0.08" rpy="0 0 0"/>
+    <axis xyz="0 1 0"/>
+    <limit velocity="6.5" effort="1000" lower="${-pi/2}" upper="${pi}" />
+    <dynamics damping = "0.7"/>
+  </joint>
+  <transmission name="r_shoulder_pitch_tran">
+     <type>transmission_interface/SimpleTransmission</type>
+     <joint name="r_shoulder_pitch">
+       <hardwareInterface>EffortJointInterface</hardwareInterface>
+     </joint>
+     <actuator name="r_shoulder_pitch_motor">
+       <hardwareInterface>EffortJointInterface</hardwareInterface>
+       <mechanicalReduction>1</mechanicalReduction>
+     </actuator>
+  </transmission>
+  <link name="r_shoulder_pitch_link">
+    <collision>
+      <origin xyz="0 0 0" rpy="0 0 0"/>
+      <geometry>
+          <mesh filename="package://alice_1_description/meshes/asm_hum_fb_3_shr_r1.stl" scale="0.001 0.001 0.001"/>
+        </geometry>
+    </collision>
+    <visual>
+        <origin xyz="0 0 0" rpy="0 0 0"/>
+        <geometry>
+          <mesh filename="package://alice_1_description/meshes/asm_hum_fb_3_shr_r1.stl" scale="0.001 0.001 0.001"/>
+        </geometry>
+        <material name="red"/>
+    </visual>
+    <inertial>
+      <origin xyz="0 0 0" rpy="0 0 0"/>
+      <mass value="1"/>
+      <inertia ixx="1.0" ixy="0.0" ixz="0.0" iyy="1.0" iyz="0.0" izz="1.0" />
+    </inertial>
+  </link>
+ <joint name="r_shoulder_roll" type="revolute">
+    <parent link="r_shoulder_pitch_link"/>
+    <child link="r_shoulder_roll_link"/>
+    <origin xyz="0 0 0" rpy="0 0 0"/>
+    <axis xyz="1 0 0"/>
+    <limit velocity="6.5" effort="1000" lower="${-pi/2}" upper="${pi}" />
+    <dynamics damping = "0.7"/>
+  </joint>
+  <transmission name="r_shoulder_roll_tran">
+     <type>transmission_interface/SimpleTransmission</type>
+     <joint name="r_shoulder_roll">
+       <hardwareInterface>EffortJointInterface</hardwareInterface>
+     </joint>
+     <actuator name="r_shoulder_roll_motor">
+       <hardwareInterface>EffortJointInterface</hardwareInterface>
+       <mechanicalReduction>1</mechanicalReduction>
+     </actuator>
+  </transmission>
+  <link name="r_shoulder_roll_link">
+    <collision>
+      <origin xyz="0 0 0" rpy="0 0 0"/>
+      <geometry>
+          <mesh filename="package://alice_1_description/meshes/prt_hum_fb_3_elbow_l.stl" scale="0.001 0.001 0.001"/>
+        </geometry>
+    </collision>
+    <visual>
+        <origin xyz="0 0 0" rpy="0 0 0"/>
+        <geometry>
+          <mesh filename="package://alice_1_description/meshes/prt_hum_fb_3_elbow_l.stl" scale="0.001 0.001 0.001"/>
+        </geometry>
+        <material name="red"/>
+    </visual>
+    <inertial>
+      <origin xyz="0 0 0" rpy="0 0 0"/>
+      <mass value="1"/>
+      <inertia ixx="1.0" ixy="0.0" ixz="0.0" iyy="1.0" iyz="0.0" izz="1.0" />
+    </inertial>
+  </link>
+ <joint name="r_elbow_pitch" type="revolute">
+    <parent link="r_shoulder_roll_link"/>
+    <child link="r_elbow_pitch_link"/>
+    <origin xyz="0 0 -0.27" rpy="0 0 0"/>
+    <axis xyz="0 -1 0"/>
+    <limit velocity="6.5" effort="1000" lower="${-pi/2}" upper="${pi}" />
+    <dynamics damping = "0.7"/>
+  </joint>
+  <transmission name="r_elbow_pitch_tran">
+     <type>transmission_interface/SimpleTransmission</type>
+     <joint name="r_elbow_pitch">
+       <hardwareInterface>EffortJointInterface</hardwareInterface>
+     </joint>
+     <actuator name="r_elbow_pitch_motor">
+       <hardwareInterface>EffortJointInterface</hardwareInterface>
+       <mechanicalReduction>1</mechanicalReduction>
+     </actuator>
+  </transmission>
+  <link name="r_elbow_pitch_link">
+    <collision>
+      <origin xyz="0 0 0" rpy="0 0 0"/>
+      <geometry>
+          <mesh filename="package://alice_1_description/meshes/prt_hum_fb_3_elbo_2_l.stl" scale="0.001 0.001 0.001"/>
+        </geometry>
+    </collision>
+    <visual>
+        <origin xyz="0 0 0" rpy="0 0 0"/>
+        <geometry>
+          <mesh filename="package://alice_1_description/meshes/prt_hum_fb_3_elbo_2_l.stl" scale="0.001 0.001 0.001"/>
+        </geometry>
+        <material name="red"/>
+    </visual>
+    <inertial>
+      <origin xyz="0 0 0" rpy="0 0 0"/>
+      <mass value="1"/>
+      <inertia ixx="1.0" ixy="0.0" ixz="0.0" iyy="1.0" iyz="0.0" izz="1.0" />
+    </inertial>
+  </link>
 <!-- head -->
 <joint name="head" type="fixed">

Commit message: axis change

File: alice_1_description/urdf/alice_1_robot.xacro (robot description, xacro)
@@ -117,5 +117,5 @@
     <child link="head_pitch_link"/>
     <origin xyz="0 0 0.023" rpy="0 0 0"/>
-    <axis xyz="0 1 0"/>
+    <axis xyz="0 -1 0"/>
     <limit velocity="6.5" effort="1000" lower="${-pi/2}" upper="${pi}" />
     <dynamics damping = "0.7"/>
@@ -314,5 +314,5 @@
     <child link="r_shoulder_pitch_link"/>
     <origin xyz="0 -0.17 0.4100" rpy="0 0 0"/>
-    <axis xyz="0 1 0"/>
+    <axis xyz="0 -1 0"/>
     <limit velocity="6.5" effort="1000" lower="${-pi/2}" upper="${pi}" />
     <dynamics damping = "0.7"/>
@@ -429,5 +429,5 @@
     <child link="l_hip_pitch_link"/>
     <origin xyz="0 0.021 0" rpy="0 0 0"/>
-    <axis xyz="0 -1 0"/>
+    <axis xyz="0 1 0"/>
     <limit velocity="6.5" effort="1000" lower="${-pi/2}" upper="${pi}" />
     <dynamics damping = "0.7"/>
@@ -467,5 +467,5 @@
     <child link="l_hip_roll_link"/>
     <origin xyz="0 0.059 0" rpy="0 0 0"/>
-    <axis xyz="-1 0 0"/>
+    <axis xyz="1 0 0"/>
     <limit velocity="6.5" effort="1000" lower="${-pi/2}" upper="${pi}" />
     <dynamics damping = "0.7"/>
@@ -666,5 +666,5 @@
     <child link="r_hip_pitch_link"/>
     <origin xyz="0 -0.021 0" rpy="0 0 0"/>
-    <axis xyz="0 1 0"/>
+    <axis xyz="0 -1 0"/>
     <limit velocity="6.5" effort="1000" lower="${-pi/2}" upper="${pi}" />
     <dynamics damping = "0.7"/>
@@ -704,5 +704,5 @@
     <child link="r_hip_roll_link"/>
     <origin xyz="0 -0.059 0" rpy="0 0 0"/>
-    <axis xyz="-1 0 0"/>
+    <axis xyz="1 0 0"/>
     <limit velocity="6.5" effort="1000" lower="${-pi/2}" upper="${pi}" />
     <dynamics damping = "0.7"/>

File: alice_2_description/urdf/alice_2_robot.xacro (robot description, xacro)
@@ -194,5 +194,5 @@
     <child link="r_shoulder_pitch_link"/>
     <origin xyz="0 -0.175 0.08" rpy="0 0 0"/>
-    <axis xyz="0 1 0"/>
+    <axis xyz="0 -1 0"/>
     <limit velocity="6.5" effort="1000" lower="${-pi/2}" upper="${pi}" />
     <dynamics damping = "0.7"/>

Commit message: head

File: alice_1_description/urdf/alice_1_robot.xacro (robot description, xacro)
@@ -117,5 +117,5 @@
     <child link="head_pitch_link"/>
     <origin xyz="0 0 0.023" rpy="0 0 0"/>
-    <axis xyz="0 -1 0"/>
+    <axis xyz="0 1 0"/>
     <limit velocity="6.5" effort="1000" lower="${-pi/2}" upper="${pi}" />
     <dynamics damping = "0.7"/>

Commit message: 1 gazebo

File: alice_1_description/urdf/alice_1_robot.xacro (robot description, xacro)
@@ -429,5 +429,5 @@
     <child link="l_hip_pitch_link"/>
     <origin xyz="0 0.021 0" rpy="0 0 0"/>
-    <axis xyz="0 1 0"/>
+    <axis xyz="0 -1 0"/>
     <limit velocity="6.5" effort="1000" lower="${-pi/2}" upper="${pi}" />
     <dynamics damping = "0.7"/>
@@ -581,5 +581,5 @@
     <child link="l_ankle_pitch_link"/>
     <origin xyz="0 0 -0.28" rpy="0 0 0"/>
-    <axis xyz="0 1 0"/>
+    <axis xyz="0 -1 0"/>
     <limit velocity="6.5" effort="1000" lower="${-pi/2}" upper="${pi}" />
     <dynamics damping = "0.7"/>
@@ -666,5 +666,5 @@
     <child link="r_hip_pitch_link"/>
     <origin xyz="0 -0.021 0" rpy="0 0 0"/>
-    <axis xyz="0 -1 0"/>
+    <axis xyz="0 1 0"/>
     <limit velocity="6.5" effort="1000" lower="${-pi/2}" upper="${pi}" />
     <dynamics damping = "0.7"/>
@@ -818,5 +818,5 @@
     <child link="r_ankle_pitch_link"/>
     <origin xyz="0 0 -0.28" rpy="0 0 0"/>
-    <axis xyz="0 -1 0"/>
+    <axis xyz="0 1 0"/>
     <limit velocity="6.5" effort="1000" lower="${-pi/2}" upper="${pi}" />
     <dynamics damping = "0.7"/>
